File: Aladdin Lamp.brd (EAGLE design)
At the start: 115 x 30 mm, 42 parts, among them IC1 74HCT125D, U1 M5STAMP PICO

Commit message: cosmetic changes
Other:
- board text added: "5V"

Commit message: final v1.0
Parts:
- added R2: 10K, Resistor:RESC2012X65
- added S2: SW, SparkFun-Switches:SWITCH_SPST_SMD_A
- J2: value (none) -> TARGET
- PWR: value (none) -> 5V5
- moved S1 2.00 mm to (27.0, 25.0), turned to 180 degrees
Connections:
- new net SW: R2.2, S2.3, U1.13
- net 3V3: now also S2.2
- net GND: now also R2.1
Routing:
- net VCC: track 675.5 -> 634.8 mm
- net SW: track 0.00 -> 28.5 mm, vias 0 -> 1
- net 3V3: track 0.00 -> 27.0 mm, vias 0 -> 1
- net TX: track 24.6 -> 16.8 mm
- net G0: track 13.1 -> 6.07 mm
- net RX: track 16.4 -> 17.0 mm
- added copper zone on layer 1, net N$1
- added copper zone on layer 1, net N$2
- added copper zone on layer 16, net N$3
- added copper zone on layer 16, net N$4
Other:
- outline, holes or cut-outs redrawn
- board text added: "Aladdin Lamp V1.0 0x76656e"
