File: Aladdin Lamp.sch (EAGLE design)
At the start: 42 parts, among them IC1 74HCT125D, U1 M5STAMP PICO

Commit message: final v1.0
Parts:
- added R2: 10K, Resistor:R-US_CHIP-0805(2012-METRIC)
- added S2: SW, SparkFun-Switches:SWITCH-SPDT-SMD-RIGHT-ANGLE
- J2: value (none) -> TARGET
- PWR: value (none) -> 5V5
Connections:
- new net 3V3: S2.P, U1.3V3
- new net SW: R2.2, S2.S, U1.G33
- net GND: now also R2.1
Changed lines of the file:
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@@
 <part name="FRAME1" library="frames" library_urn="urn:adsk.eagle:library:229" deviceset="DINA5_L" device="" value="ESP32 PICO"/>
 <part name="S1" library="SparkFun-Switches" library_urn="urn:adsk.eagle:library:535" deviceset="MOMENTARY-SWITCH-SPST" device="-SMD-5.2MM" package3d_urn="urn:adsk.eagle:package:40167/1" value="FLASH"/>
-<part name="FRAME2" library="frames" library_urn="urn:adsk.eagle:library:229" deviceset="A4L-LOC" device=""/>
+<part name="FRAME2" library="frames" library_urn="urn:adsk.eagle:library:229" deviceset="A4L-LOC" device="" value="LED"/>
 <part name="D9" library="SparkFun-LED" library_urn="urn:adsk.eagle:library:529" deviceset="APA102" device="-5050"/>
 <part name="D10" library="SparkFun-LED" library_urn="urn:adsk.eagle:library:529" deviceset="APA102" device="-5050"/>
@@
 <part name="D17" library="LED" library_urn="urn:adsk.eagle:library:22900745" deviceset="CHIP-FLAT-R" device="_0805" package3d_urn="urn:adsk.eagle:package:24294806/1" value="LED_RED"/>
 <part name="R1" library="Resistor" library_urn="urn:adsk.eagle:library:16378527" deviceset="R-US" device="CHIP-0805(2012-METRIC)" package3d_urn="urn:adsk.eagle:package:16378559/2" technology="_" value="330"/>
-<part name="PWR" library="Wurth_Connectors_WR-TBL Rising Cage Clamp" library_urn="urn:adsk.eagle:library:16280519" deviceset="691213510002" device="" package3d_urn="urn:adsk.eagle:package:16248575/2"/>
+<part name="PWR" library="Wurth_Connectors_WR-TBL Rising Cage Clamp" library_urn="urn:adsk.eagle:library:16280519" deviceset="691213510002" device="" package3d_urn="urn:adsk.eagle:package:16248575/2" value="5V5"/>
 <part name="H1" library="holes" library_urn="urn:adsk.eagle:library:237" deviceset="MOUNT-HOLE" device="2.8" package3d_urn="urn:adsk.eagle:package:14271/1"/>
 <part name="H2" library="holes" library_urn="urn:adsk.eagle:library:237" deviceset="MOUNT-HOLE" device="2.8" package3d_urn="urn:adsk.eagle:package:14271/1"/>
-<part name="J2" library="custom" library_urn="urn:adsk.eagle:library:28163416" deviceset="6_PIN_SERIAL_TARGET" device="SILK" package3d_urn="urn:adsk.eagle:package:37733454/1"/>
+<part name="J2" library="custom" library_urn="urn:adsk.eagle:library:28163416" deviceset="6_PIN_SERIAL_TARGET" device="SILK" package3d_urn="urn:adsk.eagle:package:37733454/1" value="TARGET"/>
+<part name="S2" library="SparkFun-Switches" library_urn="urn:adsk.eagle:library:535" deviceset="SWITCH-SPDT" device="-SMD-RIGHT-ANGLE" package3d_urn="urn:adsk.eagle:package:40179/1" value="SW"/>
+<part name="R2" library="Resistor" library_urn="urn:adsk.eagle:library:16378527" deviceset="R-US" device="CHIP-0805(2012-METRIC)" package3d_urn="urn:adsk.eagle:package:16378559/2" technology="_" value="10K"/>
+<part name="SUPPLY3" library="supply2" library_urn="urn:adsk.eagle:library:372" deviceset="GND" device=""/>
 </parts>
 <sheets>
@@
 <instance part="PWR" gate="G$1" x="38.1" y="93.98" smashed="yes" rot="R90">
 <attribute name="NAME" x="39.022" y="89.1" size="1.778" layer="95" rot="R180" align="bottom-right"/>
-<attribute name="VALUE" x="40.68" y="89.15" size="1.016" layer="96" rot="R90" align="bottom-right"/>
+<attribute name="VALUE" x="38.14" y="96.77" size="1.016" layer="96" rot="R180" align="bottom-right"/>
 </instance>
 <instance part="H1" gate="G$1" x="38.1" y="73.66" smashed="yes">
@@
 <attribute name="VALUE" x="136.906" y="40.64" size="1.778" layer="96" font="vector" rot="R90"/>
 <attribute name="NAME" x="116.332" y="40.64" size="1.778" layer="95" font="vector" rot="R90"/>
+</instance>
+<instance part="S2" gate="1" x="43.18" y="35.56" smashed="yes">
+<attribute name="NAME" x="44.45" y="38.608" size="1.778" layer="95" font="vector" align="bottom-center"/>
+<attribute name="VALUE" x="44.196" y="32.258" size="1.778" layer="96" font="vector" align="top-center"/>
+</instance>
+<instance part="R2" gate="G$1" x="58.42" y="33.02" smashed="yes" rot="R180">
+<attribute name="NAME" x="58.42" y="36.6014" size="1.778" layer="95" rot="R180" align="center"/>
+<attribute name="VALUE" x="58.42" y="39.37" size="1.778" layer="96" rot="R180" align="center"/>
+</instance>
+<instance part="SUPPLY3" gate="GND" x="66.04" y="20.32" smashed="yes">
+<attribute name="VALUE" x="64.135" y="17.145" size="1.778" layer="96"/>
 </instance>
 </instances>
@@
 <label x="160.02" y="96.52" size="0.8128" layer="95" xref="yes"/>
 </segment>
+<segment>
+<pinref part="R2" gate="G$1" pin="1"/>
+<wire x1="63.5" y1="33.02" x2="66.04" y2="33.02" width="0.1524" layer="91"/>
+<wire x1="66.04" y1="33.02" x2="66.04" y2="22.86" width="0.1524" layer="91"/>
+<pinref part="SUPPLY3" gate="GND" pin="GND"/>
+</segment>
 </net>
 <net name="CLK$1" class="0">
@@
 </segment>
 </net>
+<net name="SW" class="0">
+<segment>
+<pinref part="U1" gate="G$1" pin="G33"/>
+<wire x1="104.14" y1="78.74" x2="106.68" y2="78.74" width="0.1524" layer="91"/>
+<label x="106.68" y="78.74" size="0.8128" layer="95" xref="yes"/>
+</segment>
+<segment>
+<label x="45.72" y="20.32" size="0.8128" layer="95" rot="R180" xref="yes"/>
+<pinref part="R2" gate="G$1" pin="2"/>
+<pinref part="S2" gate="1" pin="S"/>
+<wire x1="53.34" y1="33.02" x2="50.8" y2="33.02" width="0.1524" layer="91"/>
+<wire x1="50.8" y1="33.02" x2="48.26" y2="33.02" width="0.1524" layer="91"/>
+<wire x1="45.72" y1="20.32" x2="50.8" y2="20.32" width="0.1524" layer="91"/>
+<wire x1="50.8" y1="20.32" x2="50.8" y2="33.02" width="0.1524" layer="91"/>
+<junction x="50.8" y="33.02"/>
+</segment>
+</net>
+<net name="3V3" class="0">
+<segment>
+<pinref part="U1" gate="G$1" pin="3V3"/>
+<wire x1="104.14" y1="63.5" x2="106.68" y2="63.5" width="0.1524" layer="91"/>
+<label x="106.68" y="63.5" size="0.8128" layer="95" xref="yes"/>
+</segment>
+<segment>
+<label x="30.48" y="35.56" size="0.8128" layer="95" rot="R180" xref="yes"/>
+<pinref part="S2" gate="1" pin="P"/>
+<wire x1="30.48" y1="35.56" x2="40.64" y2="35.56" width="0.1524" layer="91"/>
+</segment>
+</net>
